Commit message: nuovo setup

File: franka_description/robots/common/franka_arm.ros2_control.xacro (robot description, xacro)
@@ -52,28 +52,53 @@
         </joint>
       </xacro:macro>
-      <xacro:if value="${arm_prefix == 'right_'}">
-        <xacro:configure_joint joint_name="${arm_prefix}${robot_type}_joint1" initial_position="0.0"/>
-        <xacro:configure_joint joint_name="${arm_prefix}${robot_type}_joint2" initial_position="${-pi/4}"/>
-        <xacro:configure_joint joint_name="${arm_prefix}${robot_type}_joint3" initial_position="0.0"/>
-        <xacro:configure_joint joint_name="${arm_prefix}${robot_type}_joint4" initial_position="${-3*pi/4}"/>
-        <xacro:configure_joint joint_name="${arm_prefix}${robot_type}_joint5" initial_position="0.0"/>
-        <xacro:configure_joint joint_name="${arm_prefix}${robot_type}_joint6" initial_position="${pi-pi/6}"/>
-        <xacro:configure_joint joint_name="${arm_prefix}${robot_type}_joint7" initial_position="${pi/4}"/>
-        <xacro:if value="${gazebo and hand}">
-          <xacro:configure_joint joint_name="${arm_prefix}${robot_type}_finger_joint1" initial_position="0.0" />
-        </xacro:if>
+     <xacro:if value="${arm_prefix == 'right_'}">
+      <xacro:configure_joint joint_name="${arm_prefix}${robot_type}_joint1" initial_position="1.0472"/>
+      <xacro:configure_joint joint_name="${arm_prefix}${robot_type}_joint2" initial_position="0.3142"/>
+      <xacro:configure_joint joint_name="${arm_prefix}${robot_type}_joint3" initial_position="0.4887"/>
+      <xacro:configure_joint joint_name="${arm_prefix}${robot_type}_joint4" initial_position="-2.3213"/>
+      <xacro:configure_joint joint_name="${arm_prefix}${robot_type}_joint5" initial_position="-1.2566"/>
+      <xacro:configure_joint joint_name="${arm_prefix}${robot_type}_joint6" initial_position="1.5184"/>
+      <xacro:configure_joint joint_name="${arm_prefix}${robot_type}_joint7" initial_position="0.2443"/>
+      <xacro:if value="${gazebo and hand}">
+        <xacro:configure_joint joint_name="${arm_prefix}${robot_type}_finger_joint1" initial_position="0.0" />
       </xacro:if>
-      <xacro:if value="${arm_prefix == 'left_'}">
-        <xacro:configure_joint joint_name="${arm_prefix}${robot_type}_joint1" initial_position="0.0"/>
-        <xacro:configure_joint joint_name="${arm_prefix}${robot_type}_joint2" initial_position="${-pi/4}"/>
-        <xacro:configure_joint joint_name="${arm_prefix}${robot_type}_joint3" initial_position="0.0"/>
-        <xacro:configure_joint joint_name="${arm_prefix}${robot_type}_joint4" initial_position="${-3*pi/4}"/>
-        <xacro:configure_joint joint_name="${arm_prefix}${robot_type}_joint5" initial_position="0.0"/>
-        <xacro:configure_joint joint_name="${arm_prefix}${robot_type}_joint6" initial_position="${pi/2}"/>
-        <xacro:configure_joint joint_name="${arm_prefix}${robot_type}_joint7" initial_position="${pi/4}"/>
-        <xacro:if value="${gazebo and hand}">
-          <xacro:configure_joint joint_name="${arm_prefix}${robot_type}_finger_joint1" initial_position="0.0" />
-        </xacro:if>
+    </xacro:if>
+     <xacro:if value="${arm_prefix == 'left_'}">
+      <xacro:configure_joint joint_name="${arm_prefix}${robot_type}_joint1" initial_position="-0.4712"/>
+      <xacro:configure_joint joint_name="${arm_prefix}${robot_type}_joint2" initial_position="-0.7505"/>
+      <xacro:configure_joint joint_name="${arm_prefix}${robot_type}_joint3" initial_position="-0.2443"/>
+      <xacro:configure_joint joint_name="${arm_prefix}${robot_type}_joint4" initial_position="-2.5482"/>
+      <xacro:configure_joint joint_name="${arm_prefix}${robot_type}_joint5" initial_position="-0.0698"/>
+      <xacro:configure_joint joint_name="${arm_prefix}${robot_type}_joint6" initial_position="3.2463"/>
+      <xacro:configure_joint joint_name="${arm_prefix}${robot_type}_joint7" initial_position="0.7156"/>
+      <xacro:if value="${gazebo and hand}">
+        <xacro:configure_joint joint_name="${arm_prefix}${robot_type}_finger_joint1" initial_position="0.0" />
       </xacro:if>
+    </xacro:if>
+<!--
+    <xacro:if value="${arm_prefix == 'left_'}">
+  <xacro:configure_joint joint_name="${arm_prefix}${robot_type}_joint1" initial_position="0.0"/>
+  <xacro:configure_joint joint_name="${arm_prefix}${robot_type}_joint2" initial_position="${-pi/4}"/>
+  <xacro:configure_joint joint_name="${arm_prefix}${robot_type}_joint3" initial_position="0.0"/>
+  <xacro:configure_joint joint_name="${arm_prefix}${robot_type}_joint4" initial_position="${-3*pi/4}"/>
+  <xacro:configure_joint joint_name="${arm_prefix}${robot_type}_joint5" initial_position="0.0"/>
+  <xacro:configure_joint joint_name="${arm_prefix}${robot_type}_joint6" initial_position="${pi-pi/6}"/>
+  <xacro:configure_joint joint_name="${arm_prefix}${robot_type}_joint7" initial_position="${pi/4}"/>
+  <xacro:if value="${gazebo and hand}">
+    <xacro:configure_joint joint_name="${arm_prefix}${robot_type}_finger_joint1" initial_position="0.0" />
+  </xacro:if>
+</xacro:if>
+   <xacro:if value="${arm_prefix == 'right_'}">
+  <xacro:configure_joint joint_name="${arm_prefix}${robot_type}_joint1" initial_position="0.0"/>
+  <xacro:configure_joint joint_name="${arm_prefix}${robot_type}_joint2" initial_position="${-pi/4}"/>
+  <xacro:configure_joint joint_name="${arm_prefix}${robot_type}_joint3" initial_position="0.0"/>
+  <xacro:configure_joint joint_name="${arm_prefix}${robot_type}_joint4" initial_position="${-3*pi/4}"/>
+  <xacro:configure_joint joint_name="${arm_prefix}${robot_type}_joint5" initial_position="0.0"/>
+  <xacro:configure_joint joint_name="${arm_prefix}${robot_type}_joint6" initial_position="${pi/2}"/>
+  <xacro:configure_joint joint_name="${arm_prefix}${robot_type}_joint7" initial_position="${pi/4}"/>
+  <xacro:if value="${gazebo and hand}">
+    <xacro:configure_joint joint_name="${arm_prefix}${robot_type}_finger_joint1" initial_position="0.0" />
+  </xacro:if>
+</xacro:if> -->
       <xacro:macro name="general_purpose_io" params="prefix command_interface index">
         <gpio name="${arm_prefix}${prefix}">

File: franka_description/robots/common/franka_arm.xacro (robot description, xacro)
@@ -128,16 +128,43 @@
     </joint>
     <link name="${prefix}link8"/>
-     <joint name="${prefix}camera_joint" type="fixed">
+    <xacro:if value="${gazebo}">
+        <joint name="${prefix}link8_aligned_joint" type="fixed">
+        <parent link="${prefix}link8"/>
+        <child link="${prefix}link8_aligned"/>
+        <origin xyz="0 0 0" rpy="0 0 ${-pi/4}"/>
+      </joint>
+  <link name="${prefix}link8_aligned"/>
+    <joint name="${prefix}camera_joint" type="fixed">
+        <parent link="${prefix}link8_aligned"/>
+        <child link="${prefix}camera_link"/>
+        <origin xyz="0.1 0.0 0.05" rpy="0 ${-pi/2+pi/4} ${-pi}"/>
+    </joint>
+      <!-- <joint name="${prefix}camera_joint" type="fixed">
+          <parent link="${prefix}link8"/>
+          <child link="${prefix}camera_link"/>
+          <origin xyz="0 0.1 0" rpy="${pi/2} ${-pi/2} ${pi/4}"/>
+      </joint> -->
+<!--
+      <joint name="${prefix}camera_joint" type="fixed">
         <parent link="${prefix}link8"/>
         <child link="${prefix}camera_link"/>
-        <origin xyz="0 0 0.05" rpy="${pi/2} ${-pi/2} ${pi/4}"/>
-    </joint>
-    <link name="${prefix}camera_link"/>
-  <link name="${prefix}camera_link_optical" />
-  <joint name="${prefix}camera_optical_joint" type="fixed">
-    <origin xyz="0.0 0 0" rpy="${-pi/2} 0 ${-pi/2}" />
-    <parent link="${prefix}camera_link"/>
-    <child link="${prefix}camera_link_optical"/>
-  </joint>
+        <origin xyz="0.162000 -0.000000 -0.007000"
+                rpy="0.000000 -0.785398 3.141593"/>
+       </joint> -->
+<!--
+      <joint name="${prefix}camera_joint" type="fixed">
+        <parent link="${prefix}link8"/>
+        <child link="${prefix}camera_link"/>
+        <origin xyz="0.1 -0.1 0"
+                rpy="0 ${-pi/4-pi/6} ${pi}"/>
+       </joint> -->
+      <link name="${prefix}camera_link"/>
+      <link name="${prefix}camera_link_optical" />
+      <joint name="${prefix}camera_optical_joint" type="fixed">
+        <origin xyz="0.0 0 0" rpy="${-pi/2} 0 ${-pi/2}" />
+        <parent link="${prefix}camera_link"/>
+        <child link="${prefix}camera_link_optical"/>
+      </joint>
+    </xacro:if>
   </xacro:macro>
 </robot>

File: franka_gazebo_bringup/urdf/franka_arm.gazebo.xacro (robot description, xacro)
@@ -10,3 +10,5 @@
     <xacro:franka_gazebo_camera link_reference="right_fr3_camera_link"
                                 sensor_name="right_camera" gz_topic="right_camera"/>
+    <xacro:franka_gazebo_camera link_reference="left_fr3_camera_link"
+                                sensor_name="left_camera" gz_topic="left_camera"/>
 </robot>
